Commit message: update

File: Kitchen_models/models_yan/elementB_old/kitchen_assembly.urdf (robot description, URDF)
Before this commit: robot kitchen_assembly, 2 links, 1 joints
Links:
- removed link world
- link base_link: mass 316.376363075488 -> 0.1; geometry collision mesh filename=./meshes/base_link.STL; visual mesh filename=./meshes/base_link.STL
Joints:
- removed joint world_to_base

File: Kitchen_models/models_yan/elementE/refrigerator_old.urdf (robot description, URDF)
Before this commit: robot refrigerator, 4 links, 3 joints
Links:
- link base_link: mass 3.21768557939853 -> 321.768557939853
- link link1: mass 0.135487719797606 -> 13.5487719797606
- link link2: mass 0.332046785590749 -> 33.2046785590749
