Commit message: update

File: URDF_robot/segbot.urdf (robot description, URDF)
Before this commit: robot segbot, 8 links, 7 joints
Links:
- link base_caster_support_link: geometry collision mesh filename=./meshes/segbot/rmp50-castor-link.obj scale=0.0254 0.0254 0.0254; visual mesh filename=./meshes/segbot/rmp50-castor-link.obj scale=0.0254 0.0254 0.0254
- link base_link: geometry collision mesh filename=./meshes/segbot/rmp50-base-link.obj scale=0.0254 0.0254 0.0254; visual mesh filename=./meshes/segbot/rmp50-base-link.obj scale=0.0254 0.0254 0.0254
- link caster_wheel_link: geometry collision mesh filename=./meshes/segbot/rmp50-castor-wheel.obj scale=0.0254 0.0254 0.0254; visual mesh filename=./meshes/segbot/rmp50-castor-wheel.obj scale=0.0254 0.0254 0.0254
- link left_wheel_link: geometry visual mesh filename=./meshes/segbot/rmp50-left-wheel.obj scale=0.0254 0.0254 0.0254
- link plate_link: geometry collision mesh filename=./meshes/segbot/plate.obj scale=0.05 0.05 0.05; visual mesh filename=./meshes/segbot/plate.obj scale=0.05 0.05 0.05
- link right_wheel_link: geometry visual mesh filename=./meshes/segbot/rmp50-right-wheel.obj scale=0.0254 0.0254 0.0254
