Commit message: 更新代码结构

File: refactor/Asset/mobile_manipulator/arm/ur5e/ur5e_vacuum_long.urdf (robot description, URDF)
Before this commit: robot ur5e, 13 links, 12 joints
Links:
- link base_link: geometry collision mesh filename=./meshes/collision/base.stl scale=1.0 1.0 1.0; visual mesh filename=./meshes/visual/base.dae
- link forearm_link: geometry collision mesh filename=./meshes/collision/forearm.stl scale=1.0 1.0 1.0; visual mesh filename=./meshes/visual/forearm.dae
- link headLink: geometry collision mesh filename=../.././end_effector/sucker/long_vacuum_gripper/head.obj scale=0.001 0.001 0.001; visual mesh filename=../.././end_effector/sucker/long_vacuum_gripper/head.obj scale=0.001 0.001 0.001
- link lite_vacuum_gripper_link: geometry visual mesh filename=../.././end_effector/sucker/long_vacuum_gripper/base.obj scale=0.001 0.001 0.001
- link midLink: geometry visual mesh filename=../.././end_effector/sucker/long_vacuum_gripper/mid.obj scale=0.001 0.001 0.001
- link shoulder_link: geometry collision mesh filename=./meshes/collision/shoulder.stl scale=1.0 1.0 1.0; visual mesh filename=./meshes/visual/shoulder.dae
- link tipLink: geometry collision cylinder length=0.028 radius=0.001; visual mesh filename=../.././end_effector/sucker/long_vacuum_gripper/tip.obj scale=0.001 0.001 0.001
- link upper_arm_link: geometry collision mesh filename=./meshes/collision/upperarm.stl scale=1.0 1.0 1.0; visual mesh filename=./meshes/visual/upperarm.dae
- link wrist_1_link: geometry collision mesh filename=./meshes/collision/wrist1.stl scale=1.0 1.0 1.0; visual mesh filename=./meshes/visual/wrist1.dae
- link wrist_2_link: geometry collision mesh filename=./meshes/collision/wrist2.stl scale=1.0 1.0 1.0; visual mesh filename=./meshes/visual/wrist2.dae
- link wrist_3_link: geometry collision mesh filename=./meshes/collision/wrist3.stl scale=1.0 1.0 1.0; visual mesh filename=./meshes/visual/wrist3.dae

File: refactor/Asset/mobile_manipulator/base/segbot/segbot.urdf (robot description, URDF)
Before this commit: robot segbot, 8 links, 7 joints
Links:
- link base_caster_support_link: geometry collision mesh filename=./meshes/rmp50-castor-link.obj scale=0.0254 0.0254 0.0254; visual mesh filename=./meshes/rmp50-castor-link.obj scale=0.0254 0.0254 0.0254
- link base_link: geometry collision mesh filename=./meshes/rmp50-base-link.obj scale=0.0254 0.0254 0.0254; visual mesh filename=./meshes/rmp50-base-link.obj scale=0.0254 0.0254 0.0254
- link caster_wheel_link: geometry collision mesh filename=./meshes/rmp50-castor-wheel.obj scale=0.0254 0.0254 0.0254; visual mesh filename=./meshes/rmp50-castor-wheel.obj scale=0.0254 0.0254 0.0254
- link left_wheel_link: geometry visual mesh filename=./meshes/rmp50-left-wheel.obj scale=0.0254 0.0254 0.0254
- link plate_link: geometry collision mesh filename=./meshes/plate.obj scale=0.05 0.05 0.05; visual mesh filename=./meshes/plate.obj scale=0.05 0.05 0.05
- link right_wheel_link: geometry visual mesh filename=./meshes/rmp50-right-wheel.obj scale=0.0254 0.0254 0.0254
