Commit message: 更新一下机械臂的urdf文件

File: Asset/mobile_manipulator/arm/panda/panda.urdf (robot description, URDF)
Before this commit: robot panda, 13 links, 12 joints
Links:
- link panda_hand: geometry collision mesh filename=./meshes/collision/hand.obj; visual mesh filename=./meshes/visual/hand.obj
- link panda_leftfinger: geometry collision mesh filename=./meshes/collision/finger.obj; visual mesh filename=./meshes/visual/finger.obj
- link panda_link0: geometry collision mesh filename=./meshes/collision/link0.obj; visual mesh filename=./meshes/collision/link0.obj
- link panda_link1: geometry collision mesh filename=./meshes/collision/link1.obj; visual mesh filename=./meshes/visual/link1.obj
- link panda_link2: geometry collision mesh filename=./meshes/collision/link2.obj; visual mesh filename=./meshes/visual/link2.obj
- link panda_link3: geometry collision mesh filename=./meshes/collision/link3.obj; visual mesh filename=./meshes/visual/link3.obj
- link panda_link4: geometry collision mesh filename=./meshes/collision/link4.obj; visual mesh filename=./meshes/visual/link4.obj
- link panda_link5: geometry collision mesh filename=./meshes/collision/link5.obj; visual mesh filename=./meshes/visual/link5.obj
- link panda_link6: geometry collision mesh filename=./meshes/collision/link6.obj; visual mesh filename=./meshes/visual/link6.obj
- link panda_link7: geometry collision mesh filename=./meshes/collision/link7.obj; visual mesh filename=./meshes/collision/link7.obj
- link panda_rightfinger: geometry collision mesh filename=./meshes/collision/finger.obj; visual mesh filename=./meshes/visual/finger.obj

File: Asset/mobile_manipulator/arm/ur5e/ur5e_2f85.urdf (robot description, URDF)
Before this commit: robot ur5e, 20 links, 19 joints
Links:
- link base_link: geometry collision mesh filename=./meshes/collision/base.stl scale=1.0 1.0 1.0; visual mesh filename=./meshes/visual/base.dae
- link forearm_link: geometry collision mesh filename=./meshes/collision/forearm.stl scale=1.0 1.0 1.0; visual mesh filename=./meshes/visual/forearm.dae
- link shoulder_link: geometry collision mesh filename=./meshes/collision/shoulder.stl scale=1.0 1.0 1.0; visual mesh filename=./meshes/visual/shoulder.dae
- link upper_arm_link: geometry collision mesh filename=./meshes/collision/upperarm.stl scale=1.0 1.0 1.0; visual mesh filename=./meshesvisual/upperarm.dae
- link wrist_1_link: geometry collision mesh filename=./meshes/collision/wrist1.stl scale=1.0 1.0 1.0; visual mesh filename=./meshes/visual/wrist1.dae
- link wrist_2_link: geometry collision mesh filename=./meshes/collision/wrist2.stl scale=1.0 1.0 1.0; visual mesh filename=./meshes/visual/wrist2.dae
- link wrist_3_link: geometry collision mesh filename=./meshes/collision/wrist3.stl scale=1.0 1.0 1.0; visual mesh filename=./meshes/visual/wrist3.dae

File: Asset/mobile_manipulator/arm/ur5e/ur5e_vacuum.urdf (robot description, URDF)
Before this commit: robot ur5e, 10 links, 9 joints
Links:
- link base_link: geometry collision mesh filename=./meshes/collision/base.stl scale=1.0 1.0 1.0; visual mesh filename=./meshes/visual/base.dae
- link forearm_link: geometry collision mesh filename=./meshes/collision/forearm.stl scale=1.0 1.0 1.0; visual mesh filename=./meshes/visual/forearm.dae
- link lite_vacuum_gripper_link: geometry collision mesh filename=../.././end_effector/sucker/vacuum_gripper/collision/vacuum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 scale=1.0 1.0 1.0; visual mesh filename=../.././end_effector/sucker/vacuum_gripper/visual/vacuum_gr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
- link shoulder_link: geometry collision mesh filename=./meshes/collision/shoulder.stl scale=1.0 1.0 1.0; visual mesh filename=./meshes/visual/shoulder.dae
- link upper_arm_link: geometry collision mesh filename=./meshes/collision/upperarm.stl scale=1.0 1.0 1.0; visual mesh filename=./meshes/visual/upperarm.dae
- link wrist_1_link: geometry collision mesh filename=./meshes/collision/wrist1.stl scale=1.0 1.0 1.0; visual mesh filename=./meshes/visual/wrist1.dae
- link wrist_2_link: geometry collision mesh filename=./meshes/collision/wrist2.stl scale=1.0 1.0 1.0; visual mesh filename=./meshes/visual/wrist2.dae
- link wrist_3_link: geometry collision mesh filename=./meshes/collision/wrist3.stl scale=1.0 1.0 1.0; visual mesh filename=./meshes/visual/wrist3.dae
