Commit message: 更新blender渲染相关代码以及物体模型文件中部分出错的部分

File: Asset/Kitchen_models/models/Dishwasher/2085/mobility.urdf (robot description, URDF)
Before this commit: robot partnet_185cf76909e948f0fa80fb391ee7ccee, 7 links, 6 joints
Joints:
- joint dishwasher_door: limit lower=0 upper=0.712 -> lower=0 upper=0.712 effort=30 velocity=1.0

File: Asset/Kitchen_models/models/Fridge/10144/mobility.urdf (robot description, URDF)
Before this commit: robot partnet_9e53ec8bedae98859807c66948157e66, 11 links, 10 joints
Joints:
- joint frame_to_handle: limit lower=0.0 upper=0.4 effort=1000.0 -> lower=0.0 upper=0.4 effort=1000.0 velocity=1.0
- joint fridge_door: limit lower=0.0 upper=2.967 -> lower=0.0 upper=2.967 effort=30 velocity=1.0

File: Asset/Kitchen_models/models/Microwave/7128/mobility.urdf (robot description, URDF)
Before this commit: robot partnet_c75ebd7c340649ba5ad304c2564ae1df, 7 links, 6 joints
Joints:
- joint joint_0: limit lower=-0.0 upper=1.5707963267948966 -> lower=-0.0 upper=1.5707963267948966 effort=30 velocity=1.0
- joint joint_1: limit lower=0.0040000000000000036 upper=0.01200000000000001 -> lower=0.0040000000000000036 upper=0.01200000000000001 effort=30 velocity=1.0

File: Asset/Kitchen_models/models_yan/elementA/urdf/kitchen_part_right_gen_convex.urdf (robot description, URDF)
Before this commit: robot kitchen_part_right, 60 links, 59 joints
Links:
- link baker_handle: geometry collision mesh filename=../meshes/obj/handle.obj scale=1.0 1.0 1.0; visual mesh filename=../meshes/obj/handle.obj scale=1.0 1.0 1.0
- link baker_link: geometry collision mesh filename=../meshes/obj/front_vertical_right.obj scale=1.0 1.0 1.0; visual mesh filename=../meshes/obj/front_vertical_right.obj scale=1.0 1.0 1.0
- link chewie_door_left_handle: geometry collision mesh filename=../meshes/obj/handle.obj scale=1.0 1.0 1.0; visual mesh filename=../meshes/obj/handle.obj scale=1.0 1.0 1.0
- link chewie_door_left_link: geometry collision mesh filename=../meshes/obj/front_vertical_left.obj scale=1.0 1.0 1.0; visual mesh filename=../meshes/obj/front_vertical_left.obj scale=1.0 1.0 1.0
- link chewie_door_right_handle: geometry collision mesh filename=../meshes/obj/handle.obj scale=1.0 1.0 1.0; visual mesh filename=../meshes/obj/handle.obj scale=1.0 1.0 1.0
- link chewie_door_right_link: geometry collision mesh filename=../meshes/obj/front_vertical_right.obj scale=1.0 1.0 1.0; visual mesh filename=../meshes/obj/front_vertical_right.obj scale=1.0 1.0 1.0
- link dagger: geometry collision mesh filename=../meshes/obj/sektion_top_two_glass.obj scale=1.0 1.0 1.0; visual mesh filename=../meshes/obj/sektion_top_two_glass.obj scale=1.0 1.0 1.0
- link dagger_door_left_handle: geometry collision mesh filename=../meshes/obj/handle.obj scale=1.0 1.0 1.0; visual mesh filename=../meshes/obj/handle.obj scale=1.0 1.0 1.0
- link dagger_door_left_link: geometry collision mesh filename=../meshes/obj/front_vertical_left.obj scale=1.0 1.0 1.0; visual mesh filename=../meshes/obj/front_vertical_left.obj scale=1.0 1.0 1.0
- link dagger_door_right_handle: geometry collision mesh filename=../meshes/obj/handle.obj scale=1.0 1.0 1.0; visual mesh filename=../meshes/obj/handle.obj scale=1.0 1.0 1.0
- link dagger_door_right_link: geometry collision mesh filename=../meshes/obj/front_vertical_right.obj scale=1.0 1.0 1.0; visual mesh filename=../meshes/obj/front_vertical_right.obj scale=1.0 1.0 1.0
- link hitman_drawer_bottom: geometry collision box size=0.005 0.699 0.086; collision box size=0.512 0.004 0.086
- link hitman_drawer_handle_bottom: geometry collision mesh filename=../meshes/obj/handle.obj scale=1.0 1.0 1.0; visual mesh filename=../meshes/obj/handle.obj scale=1.0 1.0 1.0
- link hitman_drawer_handle_top: geometry collision mesh filename=../meshes/obj/handle.obj scale=1.0 1.0 1.0; visual mesh filename=../meshes/obj/handle.obj scale=1.0 1.0 1.0
- link hitman_drawer_top: geometry collision box size=0.005 0.699 0.086; collision box size=0.512 0.004 0.086
- link hitman_tmp: geometry collision box size=0.04 0.762 0.763; collision box size=0.61 0.019 0.763
- link indigo_door_left_link: geometry collision mesh filename=../meshes/obj/front_bottom_vertical_door.obj scale=1.0 1.0 1.0; visual mesh filename=../meshes/obj/front_bottom_vertical_door.obj scale=1.0 1.0 1.0
- link indigo_door_left_nob_link: geometry collision mesh filename=../meshes/obj/handle.obj scale=1.0 1.0 1.0; visual mesh filename=../meshes/obj/handle.obj scale=1.0 1.0 1.0
- link indigo_door_right_link: geometry collision mesh filename=../meshes/obj/front_bottom_vertical_door.obj scale=1.0 1.0 1.0; visual mesh filename=../meshes/obj/front_bottom_vertical_door.obj scale=1.0 1.0 1.0
- link indigo_door_right_nob_link: geometry collision mesh filename=../meshes/obj/handle.obj scale=1.0 1.0 1.0; visual mesh filename=../meshes/obj/handle.obj scale=1.0 1.0 1.0
- link indigo_drawer_bottom: geometry collision box size=0.004 0.699 0.086; collision box size=0.511 0.004 0.086
- link indigo_drawer_handle_bottom: geometry collision mesh filename=../meshes/obj/handle.obj scale=1.0 1.0 1.0; visual mesh filename=../meshes/obj/handle.obj scale=1.0 1.0 1.0
- link indigo_drawer_handle_top: geometry collision mesh filename=../meshes/obj/handle.obj scale=1.0 1.0 1.0; visual mesh filename=../meshes/obj/handle.obj scale=1.0 1.0 1.0
- link indigo_drawer_top: geometry collision box size=0.004 0.699 0.086; collision box size=0.511 0.004 0.086
- link indigo_tmp: geometry collision box size=0.04 0.762 0.763; collision box size=0.61 0.019 0.763
- link sektion: geometry collision mesh filename=../meshes/obj/sektion_top_three.obj scale=1.0 1.0 1.0; visual mesh filename=../meshes/obj/sektion_top_three.obj scale=1.0 1.0 1.0
