Commit message: Organize the mobile_manipulator directory and update the BestMan_sim file

File: Asset/mobile_manipulator/arm/ur5e/urdf/ur5e_vacuum_long.urdf (robot description, URDF)
Before this commit: robot ur5e, 13 links, 12 joints
Links:
- link headLink: geometry collision mesh filename=../../../end_effector/vacuum_gripper/long_vacuum_gripper/me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 scale=0.00100 0.00100 0.00100; visual mesh filename=../../../end_effector/vacuum_gripper/long_vacuum_gripper/me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 scale=0.00100 0.00100 0.00100
- link midLink: geometry visual mesh filename=../../../end_effector/vacuum_gripper/long_vacuum_gripper/me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 scale=0.00100 0.00100 0.00100
- link tipLink: geometry collision cylinder length=0.02800 radius=0.00100; visual mesh filename=../../../end_effector/vacuum_gripper/long_vacuum_gripper/me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 scale=0.00100 0.00100 0.00100
