Commit message: simple change about realman

File: Asset/mobile_manipulator/base/ranger_mini3/urdf/ranger_mini3.urdf (robot description, URDF)
Before this commit: robot ranger_mini3, 8 links, 7 joints
Links:
- removed link basket_Link
- link Link7: geometry collision mesh filename=../meshes/Link7.STL; visual mesh filename=../meshes/Link7.STL
- link arm_base: geometry collision mesh filename=../meshes/arm_base.STL; visual mesh filename=../meshes/arm_base.STL
- link base_link: geometry collision mesh filename=../meshes/base_link.STL; visual mesh filename=../meshes/base_link.STL
- link front_lidar: geometry collision mesh filename=../meshes/front_lidar.STL; visual mesh filename=../meshes/front_lidar.STL
- link head_Link: geometry collision mesh filename=../meshes/head_Link.STL; visual mesh filename=../meshes/head_Link.STL
- link head_camera: geometry collision mesh filename=../meshes/head_camera.STL; visual mesh filename=../meshes/head_camera.STL
Joints:
- removed joint basket_joint

Commit message: update about realman

File: Asset/mobile_manipulator/base/ranger_mini3/urdf/ranger_mini3.urdf (robot description, URDF)
Before this commit: robot ranger_mini3, 7 links, 6 joints
Links:
- link display_Link: geometry collision box size=0.03 0.3 0.2; visual box size=0.03 0.3 0.2
