Commit message: update about robot

File: Asset/Robot/mobile_manipulator/arm/universal/urdf/ur5e_vacuum_long.urdf (robot description, URDF)
Before this commit: robot ur5e_vacuum_long, 13 links, 12 joints
Links:
- link base_link: geometry collision mesh filename=../meshes/ur5e/base.stl scale=1.00000 1.00000 1.00000; visual mesh filename=../meshes/ur5e/base.stl scale=1.00000 1.00000 1.00000
- link forearm_link: geometry collision mesh filename=../meshes/ur5e/forearm.stl scale=1.00000 1.00000 1.00000; visual mesh filename=../meshes/ur5e/forearm.stl scale=1.00000 1.00000 1.00000
- link lite_vacuum_gripper_link: geometry visual mesh filename=../meshes/ur5e/base.stl scale=0.00100 0.00100 0.00100
- link shoulder_link: geometry collision mesh filename=../meshes/ur5e/shoulder.stl scale=1.00000 1.00000 1.00000; visual mesh filename=../meshes/ur5e/shoulder.stl scale=1.00000 1.00000 1.00000
- link upper_arm_link: geometry collision mesh filename=../meshes/ur5e/upperarm.stl scale=1.00000 1.00000 1.00000; visual mesh filename=../meshes/ur5e/upperarm.stl scale=1.00000 1.00000 1.00000
- link wrist_1_link: geometry collision mesh filename=../meshes/ur5e/wrist1.stl scale=1.00000 1.00000 1.00000; visual mesh filename=../meshes/ur5e/wrist1.stl scale=1.00000 1.00000 1.00000
- link wrist_2_link: geometry collision mesh filename=../meshes/ur5e/wrist2.stl scale=1.00000 1.00000 1.00000; visual mesh filename=../meshes/ur5e/wrist2.stl scale=1.00000 1.00000 1.00000
- link wrist_3_link: geometry collision mesh filename=../meshes/ur5e/wrist3.stl scale=1.00000 1.00000 1.00000; visual mesh filename=../meshes/ur5e/wrist3.stl scale=1.00000 1.00000 1.00000
