Commit message: update scene and model

File: Asset/Scene/Kitchen_models/models/BraiserLid/100693/mobility.urdf (robot description, URDF)
Before this commit: robot partnet_d9560bfc0c051109f54e1b6f41fdd78a, 3 links, 2 joints
Joints:
- joint handle_joint: limit lower=0 upper=0.05 -> lower=0 upper=0.05 effort=50 velocity=0.1

File: Asset/Scene/Kitchen_models/models/Faucet/14/mobility.urdf (robot description, URDF)
Before this commit: robot partnet_2781a072e2645ccdedf1aa83ea962bc0, 9 links, 8 joints
Joints:
- joint joint_faucet_0: limit lower=0.0 upper=1.5707963267948966 -> lower=0.0 upper=1.5707963267948966 effort=50 velocity=0.1
- joint joint_faucet_1: limit lower=-0.0 upper=1.5707963267948966 -> lower=-0.0 upper=1.5707963267948966 effort=50 velocity=0.1

File: Asset/Scene/Kitchen_models/models/Faucet/149/mobility.urdf (robot description, URDF)
Before this commit: robot partnet_2781a072e2645ccdedf1aa83ea962bc0, 5 links, 4 joints
Joints:
- joint joint_0: limit lower=0.0 upper=1.5707963267948966 -> lower=0.0 upper=1.5707963267948966 effort=50 velocity=0.1
- joint joint_1: limit lower=-0.0 upper=1.5707963267948966 -> lower=-0.0 upper=1.5707963267948966 effort=50 velocity=0.1

File: Asset/Scene/Kitchen_models/models/MilkBottle/4043/mobility.urdf (robot description, URDF)
Before this commit: robot partnet_e7714b3280fa7f925b2cc658332a8e03, 4 links, 3 joints
Joints:
- joint joint_2: limit lower=-0.09200000000000008 upper=0.05600000000000005 -> lower=-0.09200000000000008 upper=0.05600000000000005 effort=50 velocity=0.1

File: Asset/Scene/Kitchen_models/models/Oven/01909/mobility.urdf (robot description, URDF)
Before this commit: robot partnet_8295e45a734c059d1f3d773b4af1f0c9, 8 links, 7 joints
Joints:
- joint joint_0: limit lower=-0.0 upper=1.5707963267948966 -> lower=-0.0 upper=1.5707963267948966 effort=50 velocity=0.1
- joint knob_joint_1: limit lower=-0.0 upper=1.046666667 -> lower=-0.0 upper=1.046666667 effort=50 velocity=0.1
- joint knob_joint_2: limit lower=-0.0 upper=1.046666667 -> lower=-0.0 upper=1.046666667 effort=50 velocity=0.1
- joint knob_joint_3: limit lower=-0.0 upper=5.672320068981571 -> lower=-0.0 upper=5.672320068981571 effort=50 velocity=0.1
- joint knob_joint_4: limit lower=-6.283185307179586 upper=-0.6108652381980153 -> lower=-6.283185307179586 upper=-0.6108652381980153 effort=50 velocity=0.1
