Commit message: update

File: Asset/Robot/mobile_manipulator/base/ranger_mini_v3/urdf/ranger_mini_v3.urdf (robot description, URDF)
Before this commit: robot ranger_mini_v3, 5 links, 4 joints
Links:
- link base_link: mass 0.16272 -> 0.162715996120322; geometry collision mesh filename=../meshes/ranger_mini3.dae; visual mesh filename=../meshes/ranger_mini3.dae
- link bl_Link: mass 2.27860 -> 2.2786; geometry collision mesh filename=../meshes/ranger_mini_v3_wheel.dae; visual mesh filename=../meshes/ranger_mini_v3_wheel.dae
- link br_Link: mass 2.27860 -> 2.2786; geometry collision mesh filename=../meshes/ranger_mini_v3_wheel_right.dae; visual mesh filename=../meshes/ranger_mini_v3_wheel_right.dae
- link fl_Link: mass 2.27860 -> 2.2786; geometry collision mesh filename=../meshes/ranger_mini_v3_wheel.dae; visual mesh filename=../meshes/ranger_mini_v3_wheel.dae
- link fr_Link: mass 2.27860 -> 2.2786; geometry collision mesh filename=../meshes/ranger_mini_v3_wheel_right.dae; visual mesh filename=../meshes/ranger_mini_v3_wheel_right.dae
Joints:
- joint bl_joint: axis 0.02704 0.00000 -0.99963 -> (none); limit lower=0.00000 upper=0.00000 effort=0.00000 velocity=0.00000 -> (none); origin xyz=-0.25000 0.19000 -0.10000 rpy=-3.14159 0.00000 0.00000 -> xyz=-0.25 0.19 -0.1 rpy=3.1416 0 0; type continuous -> fixed
- joint br_joint: axis 0.00397 0.00000 -0.99999 -> (none); limit lower=0.00000 upper=0.00000 effort=0.00000 velocity=0.00000 -> (none); origin xyz=-0.25000 -0.19000 -0.10000 rpy=0.00000 0.00000 0.00000 -> xyz=-0.25 -0.19 -0.1 rpy=0 0 0; type continuous -> fixed
- joint fl_joint: axis 0.04105 0.00000 -0.99916 -> (none); limit lower=0.00000 upper=0.00000 effort=0.00000 velocity=0.00000 -> (none); origin xyz=0.25000 0.19000 -0.10000 rpy=-3.14159 0.00000 0.00000 -> xyz=0.25 0.19 -0.1 rpy=3.1416 0 0; type continuous -> fixed
- joint fr_joint: axis 0.00000 0.00000 -1.00000 -> (none); limit lower=0.00000 upper=0.00000 effort=0.00000 velocity=0.00000 -> (none); origin xyz=0.25000 -0.19000 -0.10000 rpy=0.00000 0.00000 0.00000 -> xyz=0.25 -0.19 -0.1 rpy=0 0 0; type continuous -> fixed

Commit message: update about ranger mini base

File: Asset/Robot/mobile_manipulator/base/ranger_mini_v3/urdf/ranger_mini_v3.urdf (robot description, URDF)
Before this commit: robot ranger_mini_v3, 5 links, 4 joints
Links:
- link base_link: mass 0.162715996120322 -> 0.16272; geometry collision mesh filename=../meshes/ranger_mini3.stl scale=1.00000 1.00000 1.00000; visual mesh filename=../meshes/ranger_mini3.stl scale=1.00000 1.00000 1.00000
- link bl_Link: mass 2.2786 -> 2.27860; geometry collision mesh filename=../meshes/ranger_mini_v3_wheel.stl scale=1.00000 1.00000 1.00000; visual mesh filename=../meshes/ranger_mini_v3_wheel.stl scale=1.00000 1.00000 1.00000
- link br_Link: mass 2.2786 -> 2.27860; geometry collision mesh filename=../meshes/ranger_mini_v3_wheel_right.stl scale=1.00000 1.00000 1.00000; visual mesh filename=../meshes/ranger_mini_v3_wheel_right.stl scale=1.00000 1.00000 1.00000
- link fl_Link: mass 2.2786 -> 2.27860; geometry collision mesh filename=../meshes/ranger_mini_v3_wheel.stl scale=1.00000 1.00000 1.00000; visual mesh filename=../meshes/ranger_mini_v3_wheel.stl scale=1.00000 1.00000 1.00000
- link fr_Link: mass 2.2786 -> 2.27860; geometry collision mesh filename=../meshes/ranger_mini_v3_wheel_right.stl scale=1.00000 1.00000 1.00000; visual mesh filename=../meshes/ranger_mini_v3_wheel_right.stl scale=1.00000 1.00000 1.00000
Joints:
- joint bl_joint: origin xyz=-0.25 0.19 -0.1 rpy=3.1416 0 0 -> xyz=-0.25000 0.19000 -0.10000 rpy=-3.14159 0.00000 0.00000
- joint br_joint: origin xyz=-0.25 -0.19 -0.1 rpy=0 0 0 -> xyz=-0.25000 -0.19000 -0.10000 rpy=0.00000 0.00000 0.00000
- joint fl_joint: origin xyz=0.25 0.19 -0.1 rpy=3.1416 0 0 -> xyz=0.25000 0.19000 -0.10000 rpy=-3.14159 0.00000 0.00000
- joint fr_joint: origin xyz=0.25 -0.19 -0.1 rpy=0 0 0 -> xyz=0.25000 -0.19000 -0.10000 rpy=0.00000 0.00000 0.00000

Commit message: update bug about ranger mini,Too many patches on the base

File: Asset/Robot/mobile_manipulator/base/ranger_mini_v3/urdf/ranger_mini_v3.urdf (robot description, URDF)
Before this commit: robot ranger_mini_v3, 5 links, 4 joints
Links:
- link base_link: geometry collision mesh filename=../meshes/ranger_mini3_decimate.stl scale=1.00000 1.00000 1.00000; visual mesh filename=../meshes/ranger_mini3_decimate.stl scale=1.00000 1.00000 1.00000
